Commit message: updates

File: config/arm.urdf.xacro (robot description, xacro)
@@ -2,8 +2,16 @@
 <robot xmlns:xacro="http://www.ros.org/wiki/xacro" name="arm">
     <xacro:arg name="initial_positions_file" default="initial_positions.yaml" />
+    <link name="world" />
+    <link name="flange" />
+    <joint name="fix_flange" type="fixed">
+        <parent link="world" />
+        <child link="flange" />
+    </joint>
     <!-- Import arm urdf file -->
     <xacro:include filename="$(find kalman_arm_controller)/urdf/dupsko.urdf" />
     <!-- Import control_xacro -->
     <xacro:include filename="arm.ros2_control.xacro" />
-    <xacro:arm_ros2_control name="FakeSystem" initial_positions_file="$(arg initial_positions_file)"/>
+    <!-- <xacro:arm_ros2_control name="FakeSystem" initial_positions_file="$(arg initial_positions_file)"/> -->
+    <xacro:include filename="$(find kalman_arm_controller)/ros2_control/arm.ros2_control.xacro" />
+    <xacro:arm_ros2_control name="kalman_arm" />
 </robot>

Commit message: Working collisions with servo

File: config/arm.urdf.xacro (robot description, xacro)
@@ -10,4 +10,24 @@
     <!-- Import arm urdf file -->
     <xacro:include filename="$(find kalman_arm_controller)/urdf/arm_description.urdf.xacro" />
+    <joint name="fix_colision" type="fixed">
+        <parent link="world" />
+        <child link="kalman_box" />
+    </joint>
+    <link name="kalman_box">
+        <visual>
+            <geometry>
+                <!-- <mesh filename="package://kalman_arm_controller/meshes/gripper/gripper_bottom.stl" scale="0.001 0.001 0.001"/> -->
+                <box size="1.0 1.0 0.1"/>
+            </geometry>
+        <origin rpy="0 0 0" xyz="-0.04 -0.04 -0.12"/>
+        <material name="white"/>1
+        </visual>
+        <collision>
+            <geometry>
+                <box size="1.0 1.0 0.1"/>
+            </geometry>
+        <origin rpy="0 0 0" xyz="-0.04 -0.04 -0.12"/>
+        </collision>
+    </link>
     <xacro:arm_description />
     <!-- Import control_xacro -->
